File: pcb/pcb.kicad_pcb (KiCad board)
At the start: 2 copper layers, 39.2 x 20.5 mm, 9 parts, among them J2 Conn_01x08_Pin, SW1 SW_SPST

Commit message: pcb
Parts:
- added J1: Conn_01x01_Pin, Connector:connector pin1, F.Cu at (181.3, 40.4)
- turned S2 to 180 degrees
Connections:
- J2 pad 1: 1 -> unconnected-(J2-Pin_1-Pad1)
- J2 pad 2: 2 -> unconnected-(J2-Pin_2-Pad2)
- J2 pad 3: 3 -> unconnected-(J2-Pin_3-Pad3)
- J2 pad 4: 4 -> unconnected-(J2-Pin_4-Pad4)
- J2 pad 5: 5 -> unconnected-(J2-Pin_5-Pad5)
- J2 pad 6: 6 -> unconnected-(J2-Pin_6-Pad6)
- J2 pad 7: 7 -> unconnected-(J2-Pin_7-Pad7)
- J2 pad 8: 8 -> unconnected-(J2-Pin_8-Pad8)
- S1 pad 1: unconnected-(S1-Pad1) -> GND
- S1 pad 3: 1 -> unconnected-(J2-Pin_1-Pad1)
- S1 pad 4: unconnected-(S1-Pad4) -> unconnected-(J2-Pin_1-Pad1)
- S2 pad 3: unconnected-(S2-Pad3) -> unconnected-(J2-Pin_2-Pad2)
- S3 pad 3: unconnected-(S3-Pad3) -> 3
- S3 pad 4: 3 -> unconnected-(J2-Pin_3-Pad3)
- S4 pad 1: unconnected-(S4-Pad1) -> GND
- S4 pad 3: unconnected-(S4-Pad3) -> unconnected-(J2-Pin_4-Pad4)
- S5 pad 3: 5 -> unconnected-(J2-Pin_5-Pad5)
- S6 pad 3: unconnected-(S6-Pad3) -> unconnected-(J2-Pin_6-Pad6)
- S7 pad 3: 7 -> unconnected-(J2-Pin_7-Pad7)
- S7 pad 4: unconnected-(S9-Pad4) -> unconnected-(J2-Pin_7-Pad7)
- SW1 pad 1: 8 -> unconnected-(J2-Pin_8-Pad8)
Routing:
- net unconnected-(J2-Pin_4-Pad4): track 0.00 -> 27.2 mm, vias 0 -> 1
- net 4: track 23.1 -> 0.00 mm, vias 1 -> 0
- net unconnected-(J2-Pin_1-Pad1): track 0.00 -> 23.0 mm
- net 1: track 21.1 -> 0.00 mm
- net 3: track 18.3 -> 0.00 mm, vias 2 -> 0
- net unconnected-(J2-Pin_8-Pad8): track 0.00 -> 17.5 mm, vias 0 -> 1
- net 8: track 17.5 -> 0.00 mm, vias 1 -> 0
- net unconnected-(J2-Pin_2-Pad2): track 0.00 -> 17.0 mm, vias 0 -> 1
- net unconnected-(J2-Pin_3-Pad3): track 0.00 -> 15.6 mm
- net unconnected-(J2-Pin_6-Pad6): track 0.00 -> 15.0 mm, vias 0 -> 1
- net 6: track 12.6 -> 0.00 mm, vias 1 -> 0
- net unconnected-(J2-Pin_7-Pad7): track 0.00 -> 11.5 mm
- net unconnected-(J2-Pin_5-Pad5): track 0.00 -> 9.65 mm, vias 0 -> 1
- net 2: track 8.76 -> 0.00 mm, vias 1 -> 0
- net 5: track 8.71 -> 0.00 mm
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